Commit message: namespace=base works

File: husky_description/urdf/decorations.urdf.xacro (robot description, xacro)
@@ -22,7 +22,7 @@
 -->
 <robot name="husky_decorations" xmlns:xacro="http://ros.org/wiki/xacro">
-  <xacro:macro name="husky_decorate">
+  <xacro:macro name="husky_decorate" params="extra_prefix" >
     <!-- Spawn Husky chassis -->
-    <link name="top_chassis_link">
+    <link name="${extra_prefix}top_chassis_link">
       <visual>
         <origin xyz="0 0 0" rpy="0 0 0" />
@@ -33,11 +33,11 @@
     </link>
     <!-- Attach chassis to the robot -->
-    <joint name="top_chassis_joint" type="fixed">
-      <parent link="base_link" />
-      <child link="top_chassis_link" />
+    <joint name="${extra_prefix}top_chassis_joint" type="fixed">
+      <parent link="${extra_prefix}base_link" />
+      <child link="${extra_prefix}top_chassis_link" />
     </joint>
     <xacro:if value="$(optenv HUSKY_USER_RAIL_ENABLED true)">
       <!-- Spawn user rails -->
-      <link name="user_rail_link">
+      <link name="${extra_prefix}user_rail_link">
         <visual>
           <geometry>
@@ -47,13 +47,13 @@
       </link>
       <!-- Attach user rails to base link -->
-      <joint name="user_rail" type="fixed">
+      <joint name="${extra_prefix}user_rail" type="fixed">
         <origin xyz="0.272 0 0.245" rpy="0 0 0" />
-        <parent link="base_link" />
-        <child link="user_rail_link" />
+        <parent link="${extra_prefix}base_link" />
+        <child link="${extra_prefix}user_rail_link" />
       </joint>
     </xacro:if>
     <xacro:if value="$(optenv HUSKY_FRONT_BUMPER_ENABLED true)">
       <!-- Spawn front bumper link -->
-      <link name="front_bumper_link">
+      <link name="${extra_prefix}front_bumper_link">
         <visual>
           <geometry>
@@ -63,13 +63,13 @@
       </link>
       <!-- Attach front bumper -->
-      <joint name="front_bumper" type="fixed">
+      <joint name="${extra_prefix}front_bumper" type="fixed">
         <origin xyz="0.48 0 0.091" rpy="0 0 0" />
-        <parent link="base_link" />
-        <child link="front_bumper_link" />
+        <parent link="${extra_prefix}base_link" />
+        <child link="${extra_prefix}front_bumper_link" />
       </joint>
     </xacro:if>
     <xacro:if value="$(optenv HUSKY_REAR_BUMPER_ENABLED true)">
       <!-- Spawn rear bumper link -->
-      <link name="rear_bumper_link">
+      <link name="${extra_prefix}rear_bumper_link">
         <visual>
           <geometry>
@@ -79,8 +79,8 @@
       </link>
       <!-- Attach rear bumper -->
-      <joint name="rear_bumper" type="fixed">
+      <joint name="${extra_prefix}rear_bumper" type="fixed">
         <origin xyz="-0.48 0 0.091" rpy="0 0 ${M_PI}" />
-        <parent link="base_link" />
-        <child link="rear_bumper_link" />
+        <parent link="${extra_prefix}base_link" />
+        <child link="${extra_prefix}rear_bumper_link" />
       </joint>
     </xacro:if>
@@ -88,5 +88,5 @@
       <!-- Spawn the top plate -->
       <xacro:if value="$(optenv HUSKY_LARGE_TOP_PLATE false)">
-        <link name="top_plate_link">
+        <link name="${extra_prefix}top_plate_link">
           <visual>
             <origin xyz="0 0 0" rpy="0 0 0" />
@@ -109,12 +109,12 @@
         </link>
         <!-- Attach top plate -->
-        <joint name="top_plate_joint" type="fixed">
-          <parent link="base_link" />
-          <child link="top_plate_link"/>
+        <joint name="${extra_prefix}top_plate_joint" type="fixed">
+          <parent link="${extra_prefix}base_link" />
+          <child link="${extra_prefix}top_plate_link"/>
           <origin xyz="0.0812 0 0.225" rpy="0 0 0"/>
         </joint>
       </xacro:if>
       <xacro:unless value="$(optenv HUSKY_LARGE_TOP_PLATE false)">
-        <link name="top_plate_link">
+        <link name="${extra_prefix}top_plate_link">
           <visual>
             <origin xyz="0 0 0" rpy="0 0 0" />
@@ -137,7 +137,7 @@
         </link>
         <!-- Attach top plate -->
-        <joint name="top_plate_joint" type="fixed">
-          <parent link="base_link" />
-          <child link="top_plate_link"/>
+        <joint name="${extra_prefix}top_plate_joint" type="fixed">
+          <parent link="${extra_prefix}base_link" />
+          <child link="${extra_prefix}top_plate_link"/>
           <origin xyz="0.0812 0 0.245" rpy="0 0 0"/>
         </joint>

File: husky_description/urdf/husky.urdf.xacro (robot description, xacro)
@@ -29,9 +29,9 @@
   <xacro:include filename="$(find husky_description)/urdf/accessories/sensor_arch.urdf.xacro"/>
   <xacro:include filename="$(find ur_description)/urdf/ur5.urdf.xacro" />
-  <property name="M_PI" value="3.14159"/>
+  <xacro:property name="M_PI" value="3.14159"/>
   <!-- Base Size -->
-  <property name="base_x_size" value="0.98740000" />
-  <property name="base_y_size" value="0.57090000" />
-  <property name="base_z_size" value="0.24750000" />
+  <xacro:property name="base_x_size" value="0.98740000" />
+  <xacro:property name="base_y_size" value="0.57090000" />
+  <xacro:property name="base_z_size" value="0.24750000" />
   <!-- Wheel Mounting Positions -->
   <xacro:property name="wheelbase" value="0.5120" />
@@ -41,7 +41,7 @@
   <xacro:property name="wheel_length" value="0.1143" />
   <xacro:property name="wheel_radius" value="0.1651" />
-  <xacro:macro name="husky_robot">
+  <xacro:macro name="husky_robot" params="extra_prefix" >
     <!-- Base link is the center of the robot's bottom plate -->
-    <link name="base_link">
+    <link name="${extra_prefix}base_link">
       <visual>
         <origin xyz="0 0 0" rpy="0 0 0" />
@@ -64,12 +64,12 @@
     </link>
     <!-- Base footprint is on the ground under the robot -->
-    <link name="base_footprint"/>
-    <joint name="base_footprint_joint" type="fixed">
+    <link name="${extra_prefix}base_footprint"/>
+    <joint name="${extra_prefix}base_footprint_joint" type="fixed">
       <origin xyz="0 0 ${wheel_vertical_offset - wheel_radius}" rpy="0 0 0" />
-      <parent link="base_link" />
-      <child link="base_footprint" />
+      <parent link="${extra_prefix}base_link" />
+      <child link="${extra_prefix}base_footprint" />
     </joint>
     <!-- Interial link stores the robot's inertial information -->
-    <link name="inertial_link">
+    <link name="${extra_prefix}inertial_link">
       <inertial>
         <mass value="46.034"/>
@@ -78,63 +78,63 @@
       </inertial>
     </link>
-    <joint name="inertial_joint" type="fixed">
+    <joint name="${extra_prefix}inertial_joint" type="fixed">
       <origin xyz="0 0 0" rpy="0 0 0" />
-      <parent link="base_link" />
-      <child link="inertial_link" />
+      <parent link="${extra_prefix}base_link" />
+      <child link="${extra_prefix}inertial_link" />
     </joint>
     <!-- IMU Link is the standard mounting position for the UM6 IMU.-->
     <!-- Can be modified with environment variables in /etc/ros/setup.bash -->
-    <link name="imu_link"/>
-    <joint name="imu_joint" type="fixed">
+    <link name="${extra_prefix}imu_link"/>
+    <joint name="${extra_prefix}imu_joint" type="fixed">
       <origin xyz="$(optenv HUSKY_IMU_XYZ 0.19 0 0.149)" rpy="$(optenv HUSKY_IMU_RPY 0 -1.5708 3.1416)" />
-      <parent link="base_link" />
-      <child link="imu_link" />
+      <parent link="${extra_prefix}base_link" />
+      <child link="${extra_prefix}imu_link" />
     </joint>
     <gazebo reference="imu_link">
     </gazebo>
     <!-- Husky wheel macros -->
-    <xacro:husky_wheel wheel_prefix="front_left">
+    <xacro:husky_wheel wheel_prefix="front_left" extra_prefix="${extra_prefix}" >
       <origin xyz="${wheelbase/2} ${track/2} ${wheel_vertical_offset}" rpy="0 0 0" />
     </xacro:husky_wheel>
-    <xacro:husky_wheel wheel_prefix="front_right">
+    <xacro:husky_wheel wheel_prefix="front_right" extra_prefix="${extra_prefix}" >
       <origin xyz="${wheelbase/2} ${-track/2} ${wheel_vertical_offset}" rpy="0 0 0" />
     </xacro:husky_wheel>
-    <xacro:husky_wheel wheel_prefix="rear_left">
+    <xacro:husky_wheel wheel_prefix="rear_left" extra_prefix="${extra_prefix}" >
       <origin xyz="${-wheelbase/2} ${track/2} ${wheel_vertical_offset}" rpy="0 0 0" />
     </xacro:husky_wheel>
-    <xacro:husky_wheel wheel_prefix="rear_right">
+    <xacro:husky_wheel wheel_prefix="rear_right" extra_prefix="${extra_prefix}" >
       <origin xyz="${-wheelbase/2} ${-track/2} ${wheel_vertical_offset}" rpy="0 0 0" />
     </xacro:husky_wheel>
-    <xacro:husky_decorate />
+    <xacro:husky_decorate extra_prefix="${extra_prefix}" />
     <xacro:if value="$(arg ur5_enabled)">
       <xacro:property name="reflect" value="-1" />
       <!-- Spawn arm -->
-      <xacro:ur5_robot prefix="ur5_arm_" joint_limited="true"/>
+      <xacro:ur5_robot prefix="${extra_prefix}ur5_arm_" joint_limited="true"/>
       <!-- Join arm -->
-      <joint name="ur5_arm_base" type="fixed">
-        <parent link="top_plate_link" />
-        <child link="ur5_arm_base_link" />
+      <joint name="${extra_prefix}ur5_arm_base" type="fixed">
+        <parent link="${extra_prefix}top_plate_link" />
+        <child link="${extra_prefix}ur5_arm_base_link" />
         <origin xyz="0.3058 0 0.0065" rpy="0.0 0.0 -1.57" />
       </joint>
     </xacro:if>
     <xacro:if value="$(arg laser_enabled)">
-      <sick_lms1xx_mount prefix="base" topic="scan"/>
-      <joint name="laser_mount_joint" type="fixed">
+      <sick_lms1xx_mount prefix="${extra_prefix}base" topic="scan"/>
+      <joint name="${extra_prefix}laser_mount_joint" type="fixed">
         <origin xyz="$(optenv HUSKY_LMS1XX_XYZ 0.2206 0.0 0.00635)"
                 rpy="$(optenv HUSKY_LMS1XX_RPY 0.0 0.0 0.0)" />
-        <parent link="top_plate_link" />
-        <child link="base_laser_mount" />
+        <parent link="${extra_prefix}top_plate_link" />
+        <child link="${extra_prefix}base_laser_mount" />
       </joint>
     </xacro:if>
     <xacro:if value="$(arg kinect_enabled)">
-      <xacro:sensor_arch prefix="" parent="top_plate_link">
+      <xacro:sensor_arch prefix="${extra_prefix}" parent="top_plate_link">
         <origin xyz="-0.35 0 0.51" rpy="0 0 -3.14"/>
       </xacro:sensor_arch>
-      <joint name="kinect_frame_joint" type="fixed">
+      <joint name="${extra_prefix}kinect_frame_joint" type="fixed">
         <origin xyz="$(optenv HUSKY_KINECT_XYZ 0 0 0)" rpy="$(optenv HUSKY_KINECT_RPY 0 0.18 3.14)" />
-        <parent link="sensor_arch_mount_link"/>
-        <child link="camera_link"/>
+        <parent link="${extra_prefix}sensor_arch_mount_link"/>
+        <child link="${extra_prefix}camera_link"/>
       </joint>
-      <xacro:kinect_camera prefix="camera"/>
+      <xacro:kinect_camera prefix="${extra_prefix}camera" />
     </xacro:if>
     <xacro:include filename="$(optenv HUSKY_URDF_EXTRAS empty.urdf)" />

File: husky_description/urdf/wheel.urdf.xacro (robot description, xacro)
@@ -22,6 +22,6 @@
 -->
 <robot xmlns:xacro="http://ros.org/wiki/xacro" name="husky_wheel">
-	<xacro:macro name="husky_wheel" params="wheel_prefix *joint_pose">
-		<link name="${wheel_prefix}_wheel_link">
+	<xacro:macro name="husky_wheel" params="wheel_prefix *joint_pose extra_prefix">
+		<link name="${extra_prefix}${wheel_prefix}_wheel_link">
 			<inertial>
 				<mass value="2.637" />
@@ -49,7 +49,7 @@
 			<fdir1 value="1 0 0"/>
 		</gazebo>
-		<joint name="${wheel_prefix}_wheel" type="continuous">
-			<parent link="base_link"/>
-			<child link="${wheel_prefix}_wheel_link"/>
+		<joint name="${extra_prefix}${wheel_prefix}_wheel" type="continuous">
+			<parent link="${extra_prefix}base_link"/>
+			<child link="${extra_prefix}${wheel_prefix}_wheel_link"/>
 			<xacro:insert_block name="joint_pose"/>
 			<axis xyz="0 1 0" rpy="0 0 0" />
@@ -60,5 +60,5 @@
 				<mechanicalReduction>1</mechanicalReduction>
 			</actuator>
-			<joint name="${wheel_prefix}_wheel">
+			<joint name="${extra_prefix}${wheel_prefix}_wheel">
 				<hardwareInterface>VelocityJointInterface</hardwareInterface>
 			</joint>
