Commit message: fix build

File: husky_description/urdf/description.xacro (robot description, xacro)
@@ -22,8 +22,14 @@
 -->
 <robot name="husky" xmlns:xacro="http://ros.org/wiki/xacro">
-  <xacro:arg name="laser_enabled" default="false" />
-  <xacro:arg name="ur5_enabled" default="false" />
-  <xacro:arg name="kinect_enabled" default="false" />
+  <xacro:arg name="laser_enabled" default="??laser_enabled??" />
+  <xacro:arg name="ur5_enabled" default="??ur5_enabled??" />
+  <xacro:arg name="kinect_enabled" default="?kinect_enabled??" />
+  <xacro:arg name="prefix_with_underscore" default="??prefix_with_underscore??" />
   <xacro:include filename="$(find husky_description)/urdf/husky.urdf.xacro" />
-  <xacro:husky_robot />
+  <xacro:husky_robot
+    extra_prefix="$(arg prefix_with_underscore)"
+    laser_enabled="$(arg laser_enabled)"
+    ur5_enabled="$(arg ur5_enabled)"
+    kinect_enabled="$(arg kinect_enabled)"
+    />
 </robot>

File: husky_description/urdf/husky.urdf.xacro (robot description, xacro)
@@ -41,5 +41,6 @@
   <xacro:property name="wheel_length" value="0.1143" />
   <xacro:property name="wheel_radius" value="0.1651" />
-  <xacro:macro name="husky_robot" params="extra_prefix" >
+  <xacro:macro name="husky_robot"
+    params="extra_prefix laser_enabled ur5_enabled kinect_enabled" >
     <!-- Base link is the center of the robot's bottom plate -->
     <link name="${extra_prefix}base_link">
@@ -107,5 +108,5 @@
     </xacro:husky_wheel>
     <xacro:husky_decorate extra_prefix="${extra_prefix}" />
-    <xacro:if value="$(arg ur5_enabled)">
+    <xacro:if value="${ur5_enabled}">
       <xacro:property name="reflect" value="-1" />
       <!-- Spawn arm -->
@@ -118,5 +119,5 @@
       </joint>
     </xacro:if>
-    <xacro:if value="$(arg laser_enabled)">
+    <xacro:if value="${laser_enabled}">
       <sick_lms1xx_mount prefix="${extra_prefix}base" topic="scan"/>
       <joint name="${extra_prefix}laser_mount_joint" type="fixed">
@@ -127,5 +128,5 @@
       </joint>
     </xacro:if>
-    <xacro:if value="$(arg kinect_enabled)">
+    <xacro:if value="${kinect_enabled}">
       <xacro:sensor_arch prefix="${extra_prefix}" parent="top_plate_link">
         <origin xyz="-0.35 0 0.51" rpy="0 0 -3.14"/>
@@ -138,5 +139,4 @@
       <xacro:kinect_camera prefix="${extra_prefix}camera" />
     </xacro:if>
-    <xacro:include filename="$(optenv HUSKY_URDF_EXTRAS empty.urdf)" />
   </xacro:macro>
 </robot>
